File: System Management Board/Relay Stick Fix/Relay Stick Fix/Relay Stick Fix.kicad_sch (KiCad schematic)
At the start: 10 parts, among them J1 Conn_02x04, J2 Structural Header, Q1 NMOS, SW1 SW_SPDT, U1 UCC27511ADBV

Commit message: before layout revision
Parts:
- removed J2: Structural Header, Connector_PinHeader_2.54mm:PinHeader_2x04_P2.54mm_Vertical_SMD, symbol Connector_Generic:Conn_02x04_Odd_Even
- removed JP1: Jumper_2_Open, Jumper:SolderJumper-2_P1.3mm_Open_Pad1.0x1.5mm, symbol Jumper:Jumper_2_Open
- removed SW1: SW_SPDT, Package_TO_SOT_SMD:SOT-23, symbol Switch:SW_SPDT
- removed TP1: TestPoint, TestPoint:TestPoint_Pad_D2.0mm, symbol Connector:TestPoint
- removed U1: UCC27511ADBV, Package_TO_SOT_SMD:SOT-143, symbol Driver_FET:UCC27511ADBV
- added C2: 10uF, Capacitor_SMD:C_1206_3216Metric_Pad1.33x1.80mm_HandSolder, symbol Device:C
- added H1: MountingHole_Pad, MountingHole:MountingHole_3.2mm_M3_DIN965_Pad, symbol Mechanical:MountingHole_Pad
- added R3: 0, Resistor_SMD:R_1206_3216Metric_Pad1.30x1.75mm_HandSolder, symbol Device:R
- added U1: ~, Package_SO:SOIC-8-1EP_3.9x4.9mm_P1.27mm_EP2.29x3mm, symbol SMB:LT1910
- C1: value C -> 100nF
- J1: footprint Connector_PinHeader_2.54mm:PinHeader_2x04_P2.54mm_Vertical_SMD -> Connector_PinHeader_2.54mm:PinHeader_2x06_P2.54mm_Vertical_SMD; symbol Connector_Generic:Conn_02x04_Odd_Even -> Connector_Generic:Conn_02x06_Odd_Even
- R1: value R -> 5.1k
- R2: value R -> 0
Connections:
- net 5V Bootstrap: now also U1.4 (IN)
- net GND: now also C2.2, H1.1, U1.1 (GND); no longer R2.2
- net Vbat Prot: now also J1.10 (Pin_10), J1.9 (Pin_9), C2.1, R3.1, U1.5 (V+); no longer J1.7 (Pin_7), J1.8 (Pin_8), Q1.5 (D)
- net i3: now also J1.7 (Pin_7), J1.8 (Pin_8); no longer J1.5 (Pin_5), J1.6 (Pin_6)
- net at C1.1: now also U1.2 (TIMER); no longer Q1.4 (G)
- net at R2.1: now also U1.8 (GATE)
- net Fault: now reaches R1.2
- net Fault: now also U1.3 (FAULT_[SINK])
- new net: Q1.4 (G), R2.2
- new net: Q1.5 (D), R3.2, U1.7 (Sense)
- no-connect marks 2 -> 6
Other:
- moved on the sheet: Q1
