File: System Management Board/System Management Board.kicad_sch (KiCad schematic)
At the start: 151 parts, among them IC1 SI2318CDS-T1-GE3, IC2 SI2318CDS-T1-GE3, IC3 SI2318CDS-T1-GE3, IC4 SI2318CDS-T1-GE3, IC5 SI2318CDS-T1-GE3, IC6 SI2318CDS-T1-GE3, J1 Conn_01x04_Male, J10 Conn_01x02_Male, J11 Conn_02x20_Odd_Even, J12 Conn_02x05_Top_Bottom, J13 Conn_01x04_Female, J2 Conn_01x04_Male, J3 Conn_01x02_Male, J4 PJ-063BH, J6 Conn_02x06_Counter_Clockwise, J7 Conn_02x20_Odd_Even, J8 Conn_01x02_Male, J9 Conn_01x02_Male, K1 J115F11CH5VDCS61.5U, K2 J114FL1CS165VDC.41, K3 J114FL1CS165VDC.41, SW1 SW_Push, SW2 SW_Push, U1 SC0915, U4 R1560S501B-E2-FE, U5 74HC4051, U6 MCP9700T-ETT, U7 MCP9700T-ETT

Commit message: Preparation of Files for Schematic Review v0.4
Parts:
- removed C22: 100uF, Capacitor_SMD:CP_Elec_10x12.6, symbol Device:C_Polarized
- removed C23: 0.1uF, Capacitor_SMD:C_1206_3216Metric, symbol Device:C
- removed C24, C27: 10uF, Capacitor_SMD:C_1210_3225Metric, symbol Device:C
- removed D11, D12: RED, LED_SMD:LED_1206_3216Metric, symbol Device:LED
- removed D18, D19: D5V, SMB:POWERDI5_DIO, symbol SMB:SBRT15U50SP5-13
- removed D3, D5, D6: D, Diode_SMD:D_SOD-123F, symbol Device:D
- removed F2, F3, F8: 3557-10, SMB:3557-10, symbol SMB:3557-10
- removed IC2, IC3, IC6: SI2318CDS-T1-GE3, SMB:SOT95P237X112-3N, symbol SMB:SI2318CDS-T1-GE3
- removed J2: Conn_01x04_Male, SMB:1924321, symbol Connector:Conn_01x04_Male
- removed J8, J9: Conn_01x02_Male, SMB:1843606, symbol Connector:Conn_01x02_Male
- removed K2, K3: J114FL1CS165VDC.41, SMB:Big Pads - Relay_SPDT_Schrack-RT1-16A-FormC_RM5mm, symbol SMB:J114FL1CS165VDC.41
- removed PS3: I3A4W008A033V-001-R, SMB:CONV_I3A4W008A033V-001-R, symbol SMB:I3A4W008A033V-001-R
- removed R25, R29: 220k, Resistor_SMD:R_1206_3216Metric, symbol Device:R
- removed R26, R30, R33, R7, R8: 10k, Resistor_SMD:R_1206_3216Metric, symbol Device:R
- removed RL1: EE2-5NU, SMB:EE2-5NU, symbol SMB:EE2-5NU
- removed Rup1: 7.57k, Resistor_SMD:R_1206_3216Metric, symbol Device:R
- removed TP12, TP2, TP3: TestPoint, TestPoint:TestPoint_Pad_D1.0mm, symbol Connector:TestPoint
- removed U4: R1560S501B-E2-FE, SMB:HSOP-6J, symbol SMB:R1560S501B-E2-FE
- added C30, C31, C32: 180uF, Capacitor_SMD:CP_Elec_10x12.6, symbol Device:C_Polarized
- added C33, C38, C39, C40, C43, C44: 0.1uF, Capacitor_SMD:C_0603_1608Metric, symbol Device:C
- added C34, C35, C41, C42: 10uF, Capacitor_SMD:C_1210_3225Metric, symbol Device:C
- added C36, C37, C45: 1uF, Capacitor_SMD:C_1210_3225Metric, symbol Device:C
- added D11, D6: SK220A, Diode_SMD:D_SMA, symbol Device:D_Schottky
- added D20, D21: PPS1545-3G, Package_TO_SOT_SMD:TO-277B, symbol SMB:SBRT15U50SP5-13
- added FID1, FID2, FID3: Fiducial, Fiducial:Fiducial_1mm_Mask2mm, symbol Mechanical:Fiducial
- added JP5, JP6: Jmp_2_Bridged, Jumper:SolderJumper-2_P1.3mm_Bridged_RoundedPad1.0x1.5mm, symbol Jumper:SolderJumper_2_Bridged
- added L1: SRR1208-470YL, Inductor_SMD:L_Bourns_SRR1208_12.7x12.7mm, symbol Device:L
- added L2: TYS5040220M-10, Inductor_SMD:L_Bourns_SRR1208_12.7x12.7mm, symbol Device:L
- added Q2, Q3, Q4: 2N7002, Package_TO_SOT_SMD:SOT-23, symbol Transistor_FET:2N7002
- added Q5: NMOS, Package_SO:PowerPAK_SO-8L_Single, symbol Transistor_FET:CSD18543Q3A
- added R43, R45, R49: 10k, Resistor_SMD:R_0603_1608Metric, symbol Device:R
- added R44: 300k, Resistor_SMD:R_0603_1608Metric, symbol Device:R
- added R46, R47: 100k, Resistor_SMD:R_0603_1608Metric, symbol Device:R
- added R48: 54k9, Resistor_SMD:R_0603_1608Metric, symbol Device:R
- added R50: 0, Resistor_SMD:R_0603_1608Metric, symbol Device:R
- added U10, U8: LV2862YDDC, Package_TO_SOT_SMD:SOT-23-6, symbol Regulator_Switching:LV2862YDDC
- added U3: MCP1416RT-E/OT, Package_TO_SOT_SMD:SOT-23-5, symbol Driver_FET:MCP1416R
- added U4: MCP1793T-5002H/OT, Package_TO_SOT_SMD:SOT-23-5, symbol Regulator_Linear:MCP1802x-xx02xOT
- C13, C14, C19: footprint Capacitor_SMD:C_1206_3216Metric -> Capacitor_SMD:C_0603_1608Metric
- C17, C18: footprint Capacitor_SMD:C_1210_3225Metric -> Capacitor_SMD:C_0603_1608Metric
- D1, D2: value D_TVS -> SMAJ51CA
- D10, D13, D14, D15, D16, D17: value RED -> LTST-C150KRKT
- D4, D7, D8, D9: value D -> SMD26PL-TP
- F10: value Fuse -> SF-1206SA250M-2
- F6, F7: value Fuse -> 0678L9250-02
- IC1, IC4, IC5: DESCRIPTION Vishay SI2318CDS-T1-GE3 N-channel MOSFET Transistor, 5.6 A,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 -> (none)
- J1: value Conn_01x04_Male -> 200241-1112; footprint SMB:1924321 -> SMB:Molex_Mega-Fit_20024-11112_2x01_P5.70mm_Vertical; symbol Connector:Conn_01x04_Male -> Connector:Conn_01x02_Pin; Family (none) -> Mega-Fit
- J10: value Conn_01x02_Male -> 43650-0228; footprint SMB:1843606 -> Connector_Molex:Molex_Micro-Fit_3.0_43650-0215_1x02_P3.00mm_Vertical; Family (none) -> Micro-Fit
- J11: value Conn_02x20_Odd_Even -> PPPC202LFBN-RC
- J12: value Conn_02x05_Top_Bottom -> PPPC052LFBN-RC
- J13: value Conn_01x04_Female -> 43650-0415; footprint Connector_PinHeader_2.54mm:PinHeader_1x04_P2.54mm_Vertical -> Connector_Molex:Molex_Micro-Fit_3.0_43650-0415_1x04_P3.00mm_Vertical; symbol Connector:Conn_01x04_Female -> Connector:Conn_01x04_Pin; Family (none) -> Micro-Fit
- J3: value Conn_01x02_Male -> 43650-0415; footprint SMB:1843606 -> Connector_Molex:Molex_Micro-Fit_3.0_43650-0415_1x04_P3.00mm_Vertical; symbol Connector:Conn_01x02_Male -> Connector:Conn_01x04_Pin; Family (none) -> Micro-Fit
- J7: value Conn_02x20_Odd_Even -> XG4A-4035
- K1: Coil Current (none) -> Coil 300mA; Coil Voltage (none) -> Coil 5V
- R1, R10, R11, R12, R13, R14, R15, R16, R17, R18, R19, R20, R21, R22, R23, R24, R27, R28, R3, R31, R32, R34, R35, R36, R37, R38, R39, R4, R6, R9: footprint Resistor_SMD:R_1206_3216Metric -> Resistor_SMD:R_0603_1608Metric
- SW1, SW2: footprint SMB:SW_TL3305BF260QG -> Button_Switch_SMD:SW_SPST_TL3305B; symbol SMB:SW_Push_4_PIN -> Switch:SW_Push
Connections:
- net Light B Relay EN is gone; now on net LED_GREEN: U1.6 (GP4)
- net 48V Aux PWR OUT PROT: now also J3.1 (Pin_1)
- net 5V BOOTSTRAP: now also U3.3 (IN), U4.5 (VOUT)
- net 5V Logic PWR: now also D20.3
- net 5V Relay PWR: now also D21.3
- net Aux_SW: no longer J13.2 (Pin_2)
- net GND: now also J3.2 (Pin_2), J3.3 (Pin_3), TP10.1, C30.2, C31.2, C32.2, C34.2, C35.2, C36.2, C37.2, C38.2, C39.2, C40.2, C41.2, C42.2, C44.2, C45.2, D11.2 (A), D6.2 (A), JP5.1 (A), JP6.1 (A), Q2.2 (S), Q3.2 (S), Q4.2 (S), R43.2, R45.2, R49.2, U10.2 (GND), U3.2 (GND), U4.2 (GND), U8.2 (GND); no longer J1.2 (Pin_2), J13.1 (Pin_1), J3.1 (Pin_1)
- net PICO 3V3: now also C38.1, C39.1, C40.1
- net SWITCH PWR OUT PROT: now also J3.4 (Pin_4); no longer J3.2 (Pin_2)
- net Switched PWR IN PROT: now also U4.3 (~{SHDN})
- net V_batt+: now also J1.2 (Pin_2); no longer J1.3 (Pin_3), J1.4 (Pin_4)
- net V_batt+ PROT: now also C44.1, C45.1, Q5.5 (D), U3.5 (Vdd), U4.1 (VIN); no longer F10.1
- net LED_GREEN: now reaches R32.1
- net LED_GREEN: now also Q2.1 (G)
- net +24V: now reaches F10.2
- net +24V: now also C36.1, C37.1, L1.2, R44.1; no longer J13.3 (Pin_3)
- net at D9.1 (K), U1.39 (VSYS): now also C30.1, C31.1, C32.1
- net 15v PWR renamed +15V
- net 48V PWR renamed +48V
- net +48V: now also C34.1, C35.1, R46.1, U8.5 (VIN)
- net Ext_Relay_LOW_SIDE renamed BLACK_WIRE
- net BLACK_WIRE: now also F10.1
- net Ext_Relay_Trig renamed LED_RED
- net LED_RED: now also Q4.1 (G), R43.1; no longer R39.1
- net Light A Relay EN renamed LED_YELLOW
- net LED_YELLOW: now also R39.1, Q3.1 (G)
- net Light_A_Vout MES_ADC: no longer names the net of R17.1
- net Light_A_Vout MES_ADC: now also JP5.2 (B); no longer TP10.1
- net Light_B_Vout MES_ADC: no longer names the net of R18.1
- net Light_B_Vout MES_ADC: now also JP6.2 (B)
- new net: R50.1, U3.4 (OUT)
- new net: Q5.4 (G), R50.2
- new net: C33.2, D6.1 (K), L1.1, U8.6 (SW)
- new net: C43.1, U10.1 (CB)
- new net: C43.2, D11.1 (K), L2.1, U10.6 (SW)
- new net: C42.1, D20.1, D20.2, D21.1, D21.2, L2.2, R48.1
- new net: R48.2, R49.1, U10.3 (FB)
- new net: R46.2, U8.4 (~{SHDN})
- new net: C41.1, Q5.1 (S), Q5.2 (S), Q5.3 (S), R47.1, U10.5 (VIN)
- new net: C33.1, U8.1 (CB)
- new net: R44.2, R45.1, U8.3 (FB)
- new net: R47.2, U10.4 (~{SHDN})
- new net BLUE_WIRE: J13.3 (Pin_3), Q2.3 (D)
- new net BROWN_WIRE: J13.1 (Pin_1), Q4.3 (D)
- new net WHITE_WIRE: J13.2 (Pin_2), Q3.3 (D)
- no-connect marks 19 -> 15
Other:
- note added: "--Change log from rev 0.3-- Removed light bank relay A (F2, K2, D5, IC2, R7, D11, R32) Removed light bank relay B (F3, K3, D6, IC3, R8, D12, R33) Removed connector J2, J8, J9 Changed J10 to a 2 pin Molex Micro-Fit Changed J3 to a 4 pin Molex Micro-Fit Changed J13 to a 4 pin Molex Micro-Fit Remove External relay circuit (IC6) Added external status light 3 colors circuit Changed U4 from R1560S501B-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"
- note added: "Added new functions GP14 LED RED GP3 LED_YELLOW GP4 LED_GREEN"
- note added: "Barrel or Molex?"
- note added: "Buck Regulator 5V 600mA"
- note added: "External LED status light DC24V input 0.02A Red | 0.02A Yellow | 0.01A Green 4 wires #1 brown wire = Red LED #2 white wire = Yellow LED #3 blue wire = Green LED #4 black wire = Common line DC24V"
- note added: "External Status Light"
- note added: "External Status Light Power Supply 24V"
- note added: "Green Earth Wire?"
- note added: "Keep?"
- note added: "MOSFET Driver"
- note added: "Vout = 0.765V (1+ (R1 / R2))"
- note removed: "15A"
- note removed: "15V Aux PWR Out"
- note removed: "16A Lighting relays"
- note removed: "Ext Relay Driver"
- note removed: "Exterior Aux Interface Header"
- note removed: "Indicator LEDs"
- note removed: "Lighting Bank A & B"
- note removed: "PSU Enables"
- note removed: "Rup = [ Vref*F / [ Vout - Vonom]] - G Rup = [ 0.6*36500 / [ 5 - 2.59]] - 511 5V -> 8570 Ohm *5.3V -> 7570 Ohm 5.5V -> 7014 Ohm We selected a 7500 Ohm resistor to order"
- note removed: "Testing Points"
- moved on the sheet: C1, C10, C11, C12, C13, C14, C15, C16, C17, C18, C19, C2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
